Commit message: adding transparency to quadruped

File: src/dynamics/quadruped/mesh/a1.urdf (robot description, URDF)
Before this commit: robot a1_description, 23 links, 22 joints
Links:
- link FL_calf: geometry collision box size=0.2 0.016 0.016; visual mesh filename=package://mesh/calf.obj scale=1 1 1
- link FL_hip: geometry collision cylinder length=0.04 radius=0.046; visual mesh filename=package://mesh/hip.obj scale=1 1 1
- link FL_thigh: geometry collision box size=0.2 0.0245 0.034; visual mesh filename=package://mesh/thigh.obj scale=1 1 1
- link FR_calf: geometry collision box size=0.2 0.016 0.016; visual mesh filename=package://mesh/calf.obj scale=1 1 1
- link FR_hip: geometry collision cylinder length=0.04 radius=0.046; visual mesh filename=package://mesh/hip.obj scale=1 1 1
- link FR_thigh: geometry collision box size=0.2 0.0245 0.034; visual mesh filename=package://mesh/thigh_mirror.obj scale=1 1 1
- link RL_calf: geometry collision box size=0.2 0.016 0.016; visual mesh filename=package://mesh/calf.obj scale=1 1 1
- link RL_hip: geometry collision cylinder length=0.04 radius=0.046; visual mesh filename=package://mesh/hip.obj scale=1 1 1
- link RL_thigh: geometry collision box size=0.2 0.0245 0.034; visual mesh filename=package://mesh/thigh.obj scale=1 1 1
- link RR_calf: geometry collision box size=0.2 0.016 0.016; visual mesh filename=package://mesh/calf.obj scale=1 1 1
- link RR_hip: geometry collision cylinder length=0.04 radius=0.046; visual mesh filename=package://mesh/hip.obj scale=1 1 1
- link RR_thigh: geometry collision box size=0.2 0.0245 0.034; visual mesh filename=package://mesh/thigh_mirror.obj scale=1 1 1
- link trunk: geometry collision box size=0.267 0.194 0.114; visual mesh filename=package://mesh/trunk.obj scale=1 1 1
