Commit message: flamingo urdf updated

File: src/dynamics/flamingo/mesh/flamingo.urdf (robot description, URDF)
Before this commit: robot spring_flamingo, 37 links, 36 joints
Links:
- link left_foot: geometry visual box size=.01 .025 .23
- link left_strut_1: geometry visual box size=0.05 0.24 0.385
- link left_strut_10: geometry visual box size=0.05 0.23 0.385
- link left_strut_11: geometry visual box size=0.05 0.24 0.385
- link left_strut_12: geometry visual box size=0.05 0.23 0.385
- link left_strut_13: geometry visual box size=0.05 0.24 0.385
- link left_strut_14: geometry visual box size=0.05 0.23 0.385
- link left_strut_15: geometry visual box size=0.05 0.24 0.385
- link left_strut_2: geometry visual box size=0.05 0.23 0.385
- link left_strut_3: geometry visual box size=0.05 0.24 0.385
- link left_strut_4: geometry visual box size=0.05 0.23 0.385
- link left_strut_5: geometry visual box size=0.05 0.24 0.385
- link left_strut_6: geometry visual box size=0.05 0.23 0.385
- link left_strut_7: geometry visual box size=0.05 0.24 0.385
- link left_strut_8: geometry visual box size=0.05 0.23 0.385
- link left_strut_9: geometry visual box size=0.05 0.24 0.385
- link right_foot: geometry visual box size=.01 .025 .23
Joints:
- joint left_fan_fixed_joint: origin xyz=0 -0.12 0 rpy=0 0 0 -> xyz=0 0.0 0 rpy=0 0 0

Commit message: flamingo visuals

File: src/dynamics/flamingo/mesh/flamingo.urdf (robot description, URDF)
Before this commit: robot spring_flamingo, 37 links, 36 joints
Links:
- added link body, mass 0.0
Joints:
- added joint orientation: type continuous, parent body, child base_link, origin xyz=0 0.0 0 rpy=0 0 0, axis 0 1 0
